File: doc/analyze_remocon/analyze_remocon.brd (EAGLE design)
At the start: 58.1 x 27.9 mm, 20 parts, among them IC3 PIC18F2550_28DIP, Q2 BUZ11BV, X1 MINI-USB-UX60-MB-5S8

Commit message: update circuit diagram documents
Parts:
- removed C1: (no value), rcl:C0603K
- added C3: (no value), rcl:C025-025X050
- moved R9 9.16 mm to (26.7, 7.62)
- moved R8 8.98 mm to (16.5, 2.54), turned to 0 degrees
- moved R7 8.03 mm to (27.9, 11.4)
- moved R6 7.62 mm to (25.4, 11.4)
- moved R1 5.68 mm to (49.5, 5.08), turned to 180 degrees
- moved LED1 2.54 mm to (24.1, 2.54), turned to 180 degrees
- moved R10 2.54 mm to (6.35, 2.54), turned to 180 degrees
- moved LED2 2.54 mm to (29.2, 2.54)
- moved SW1 1.27 mm to (52.1, 5.08)
- moved SW2 1.27 mm to (52.1, 22.9)
Connections:
- removed net N$3: R1.1, SW1.3
- removed net N$5: R2.1, SW2.3
- removed net N$6: IC3.25, SW2.4
- new net N$7: IC3.25, R2.1, SW2.3
- net BLOCK: now also C3.1; no longer C1.1
- net GND: now also C3.2, SW2.1; no longer C1.2
- net N$4: now also R1.1
Routing:
- net N$4: track 0.00 -> 62.0 mm, vias 0 -> 1
- net BLOCK: track 85.8 -> 135.4 mm, vias 1 -> 2
- net N$7: track 0.00 -> 43.8 mm, vias 0 -> 2
- net N$6: track 32.3 -> 0.00 mm
- net GND: track 138.5 -> 164.2 mm, vias 2 -> 9
- net N$13: track 0.00 -> 7.62 mm
- net N$11: track 0.00 -> 7.62 mm
- net N$15: track 2.54 -> 7.62 mm
- net N$2: track 12.8 -> 16.0 mm
- net N$9: track 0.00 -> 2.54 mm
- net N$12: track 0.00 -> 2.54 mm
- net N$14: track 31.1 -> 29.5 mm
- net N$19: track 16.3 -> 17.8 mm, vias 0 -> 2
- net N$18: track 6.13 -> 5.08 mm
- net N$17: track 15.9 -> 15.2 mm, vias 1 -> 0

Commit message: update circuit diagram documents
Parts:
- removed C3: (no value), rcl:C025-025X050
- removed R8, R9: (no value), rcl:0207/7
- added C1: 0.1uF, rcl:C025-024X044
- added R3, R4: 1KΩ, rcl:MINI_MELF-0102R
- 2SK2201: value BUZ11BV -> (none)
- C2: value (none) -> 0.1uF; device rcl:C0603K -> rcl:C025-024X044
- IRLED1, IRLED2: value (none) -> TLN105B
- R1, R2: value (none) -> 10KΩ
- R5: value (none) -> 1Ω
- R6, R7: value (none) -> 10KΩ; device rcl:MINI_MELF-0102R -> rcl:0207/7
- RESONATOR: value (none) -> 20MHz
- moved R6 12.6 mm to (16.5, 2.54), flipped to the top, turned to 0 degrees
- moved X1 5.08 mm to (64.1, 14.0)
- moved R1 5.08 mm to (54.6, 5.08)
- moved SW1 5.08 mm to (57.1, 5.08)
- moved SW2 5.08 mm to (57.1, 22.9)
- moved R7 4.02 mm to (26.7, 7.62), flipped to the top, turned to 180 degrees
- moved R2 4.02 mm to (59.7, 22.9), turned to 0 degrees
- flipped C2 to the top, turned to 180 degrees
- renumbered IRLED to IRLED2, Q2 to 2SK2201, R10 to R5, U$1 to PL-IRM2161-C438, Y1 to RESONATOR
Connections:
- net BLOCK: now also C1.1; no longer C3.1
- net GND: now also C1.2, R6.1; no longer C3.2, R8.1
- net N$11: now also R3.1; no longer R6.1
- net N$12: now also R4.2; no longer R7.2
- net N$13: now also R4.1; no longer R7.1
- net N$14: now also R6.2, R7.1; no longer R8.2, R9.1
- net N$18: now also R7.2; no longer R9.2
- net N$9: now also R3.2; no longer R6.2
Routing:
- net N$7: track 43.8 -> 49.3 mm
- net N$4: track 62.0 -> 67.1 mm
- net N$1: track 16.4 -> 21.4 mm
- net BLOCK: track 135.4 -> 137.5 mm
- net N$2: track 16.0 -> 13.9 mm
- net GND: track 164.2 -> 165.0 mm, vias 9 -> 8
Other:
- board size 58.1 x 27.9 mm -> 63.2 x 27.9 mm

Commit message: update circuit diagram documents
Connections:
- net GND: no longer SW2.1
Routing:
- net BLOCK: track 137.5 -> 150.8 mm
- net N$2: track 13.9 -> 23.9 mm, vias 1 -> 2
- net GND: track 165.0 -> 171.6 mm, vias 8 -> 10
- net N$7: track 49.3 -> 42.9 mm
- net N$1: track 21.4 -> 27.7 mm, vias 1 -> 2
- net N$4: track 67.1 -> 66.3 mm
Changed lines of the file:
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@@
 <wire x1="0" y1="27.93" x2="0" y2="0" width="0" layer="21"/>
 <rectangle x1="12.065" y1="17.145" x2="46.355" y2="20.955" layer="41"/>
-<hole x="53.34" y="17.78" drill="0.6"/>
-<hole x="53.34" y="17.78" drill="0.6"/>
-<hole x="53.34" y="22.86" drill="0.6"/>
-<hole x="53.34" y="12.7" drill="0.6"/>
 <rectangle x1="6.985" y1="4.445" x2="14.605" y2="13.335" layer="41"/>
 <rectangle x1="31.75" y1="13.335" x2="38.735" y2="13.97" layer="41"/>
@@
 <hole x="2.54" y="15.24" drill="0.6"/>
 <rectangle x1="-5.08" y1="0" x2="0" y2="27.94" layer="16"/>
+<hole x="48.26" y="22.86" drill="0.6"/>
+<hole x="48.26" y="5.08" drill="0.6"/>
 </plain>
 <attributes>
@@
 <contactref element="R2" pad="2"/>
 <contactref element="R5" pad="2"/>
-<wire x1="55.485" y1="12.37" x2="53.34" y2="12.37" width="0.4064" layer="1"/>
-<wire x1="53.34" y1="12.37" x2="53.34" y2="12.7" width="0.4064" layer="1"/>
-<wire x1="53.34" y1="12.7" x2="55.88" y2="12.7" width="0.4064" layer="16"/>
-<via x="53.34" y="12.7" extent="1-16" drill="0.6" shape="square"/>
-<wire x1="55.88" y1="22.86" x2="55.88" y2="12.7" width="0.4064" layer="16"/>
+<wire x1="55.485" y1="12.37" x2="52.705" y2="10.465" width="0.4064" layer="1"/>
+<wire x1="52.705" y1="10.465" x2="48.26" y2="7.62" width="0.4064" layer="1"/>
+<wire x1="48.26" y1="7.62" x2="50.8" y2="7.62" width="0.4064" layer="16"/>
+<wire x1="50.8" y1="7.62" x2="50.8" y2="10.16" width="0.4064" layer="16"/>
+<via x="48.26" y="7.62" extent="1-16" drill="0.6" shape="square"/>
+<wire x1="55.88" y1="22.86" x2="55.88" y2="10.16" width="0.4064" layer="16"/>
+<wire x1="55.88" y1="10.16" x2="55.88" y2="5.08" width="0.4064" layer="16"/>
 <wire x1="2.54" y1="2.54" x2="2.54" y2="15.24" width="0.4064" layer="16"/>
 <wire x1="2.54" y1="15.24" x2="2.54" y2="20.32" width="0.4064" layer="16"/>
@@
 <wire x1="2.54" y1="20.32" x2="33.02" y2="20.32" width="0.254" layer="16"/>
 <wire x1="55.51" y1="5.08" x2="55.88" y2="5.08" width="0.4064" layer="16"/>
-<wire x1="55.88" y1="5.08" x2="55.88" y2="12.7" width="0.4064" layer="16"/>
-<wire x1="53.34" y1="12.7" x2="52.705" y2="12.7" width="0.4064" layer="1"/>
-<wire x1="52.705" y1="12.7" x2="46.355" y2="13.97" width="0.4064" layer="1" curve="-90"/>
+<wire x1="48.26" y1="7.62" x2="46.355" y2="13.97" width="0.4064" layer="1" curve="-90"/>
 <wire x1="46.355" y1="13.97" x2="43.18" y2="17.145" width="0.4064" layer="1" curve="90"/>
 <wire x1="43.18" y1="17.145" x2="9.525" y2="17.145" width="0.4064" layer="1"/>
@@
 <wire x1="33.02" y1="22.86" x2="33.02" y2="25.4" width="0.4064" layer="16"/>
 <wire x1="55.88" y1="22.86" x2="58.79" y2="22.86" width="0.4064" layer="16"/>
+<wire x1="50.8" y1="10.16" x2="55.88" y2="10.16" width="0.4064" layer="16"/>
 </signal>
 <signal name="GND">
@@
 <wire x1="53.34" y1="2.8194" x2="53.34" y2="2.54" width="0.4064" layer="16"/>
 <wire x1="43.18" y1="2.54" x2="53.34" y2="2.54" width="0.4064" layer="16"/>
-<contactref element="SW2" pad="1"/>
-<wire x1="60.4012" y1="20.5994" x2="60.6806" y2="20.32" width="0.4064" layer="16" curve="90"/>
-<wire x1="60.6806" y1="20.32" x2="60.96" y2="20.32" width="0.4064" layer="16"/>
-<wire x1="60.6806" y1="20.32" x2="58.42" y2="20.32" width="0.4064" layer="16"/>
+<wire x1="60.96" y1="20.32" x2="58.42" y2="20.32" width="0.4064" layer="16"/>
 <wire x1="58.42" y1="20.32" x2="58.42" y2="2.54" width="0.4064" layer="16"/>
 <wire x1="58.42" y1="2.54" x2="53.34" y2="2.54" width="0.4064" layer="16"/>
@@
 <contactref element="C1" pad="2"/>
 <wire x1="35.56" y1="22.86" x2="35.56" y2="25.4" width="0.4064" layer="16"/>
-<wire x1="60.96" y1="20.32" x2="53.34" y2="20.32" width="0.254" layer="1"/>
-<wire x1="53.34" y1="20.32" x2="53.8988" y2="20.5994" width="0.254" layer="1"/>
-<wire x1="60.96" y1="20.32" x2="60.4012" y2="20.5994" width="0.254" layer="1"/>
-<wire x1="53.34" y1="20.32" x2="55.485" y2="15.57" width="0" layer="19" extent="1-1"/>
+<wire x1="53.34" y1="20.32" x2="53.8988" y2="20.5994" width="0.254" layer="16"/>
+<wire x1="55.485" y1="15.57" x2="51.435" y2="16.84" width="0.4064" layer="1"/>
+<wire x1="51.435" y1="16.84" x2="48.26" y2="17.78" width="0.4064" layer="1"/>
+<wire x1="48.26" y1="17.78" x2="53.34" y2="17.78" width="0.4064" layer="16"/>
+<wire x1="53.34" y1="17.78" x2="53.34" y2="20.32" width="0.4064" layer="16"/>
+<via x="48.26" y="17.78" extent="1-16" drill="0.6" shape="square"/>
+<via x="53.34" y="20.32" extent="1-16" drill="0.6" shape="square"/>
+<wire x1="58.42" y1="20.32" x2="53.8988" y2="20.5994" width="0" layer="19" extent="16-16"/>
 </signal>
 <signal name="N$1">
 <contactref element="IC3" pad="16"/>
 <contactref element="X1" pad="2"/>
-<wire x1="52.07" y1="13.97" x2="48.26" y2="13.97" width="0.4064" layer="1"/>
-<wire x1="48.26" y1="13.97" x2="48.26" y2="17.78" width="0.4064" layer="1"/>
-<wire x1="48.26" y1="17.78" x2="43.18" y2="17.78" width="0.4064" layer="16"/>
-<wire x1="43.18" y1="17.78" x2="43.18" y2="22.86" width="0.4064" layer="16"/>
-<via x="48.26" y="17.78" extent="1-16" drill="0.6"/>
+<wire x1="48.26" y1="10.16" x2="46.99" y2="11.43" width="0.4064" layer="1" curve="-90"/>
+<wire x1="46.99" y1="11.43" x2="46.99" y2="16.51" width="0.4064" layer="1"/>
+<wire x1="46.99" y1="16.51" x2="44.45" y2="20.32" width="0.4064" layer="1"/>
+<wire x1="44.45" y1="20.32" x2="44.45" y2="24.13" width="0.4064" layer="1"/>
+<wire x1="44.45" y1="24.13" x2="43.18" y2="25.4" width="0.4064" layer="1" curve="90"/>
+<wire x1="43.18" y1="25.4" x2="43.18" y2="22.86" width="0.4064" layer="16"/>
 <wire x1="55.32" y1="13.335" x2="55.485" y2="13.17" width="0.4064" layer="1" curve="-90"/>
-<wire x1="55.32" y1="13.335" x2="53.34" y2="13.335" width="0.4064" layer="1"/>
-<wire x1="53.34" y1="13.335" x2="52.07" y2="13.97" width="0.4064" layer="1"/>
+<wire x1="48.26" y1="10.16" x2="52.945" y2="12.065" width="0.4064" layer="1"/>
+<wire x1="52.945" y1="12.065" x2="55.485" y2="13.17" width="0.4064" layer="1"/>
+<via x="48.26" y="10.16" extent="1-16" drill="0.6" shape="square"/>
+<via x="43.18" y="25.4" extent="1-16" drill="0.6" shape="square"/>
 </signal>
 <signal name="N$2">
 <contactref element="IC3" pad="15"/>
 <contactref element="X1" pad="3"/>
-<wire x1="55.245" y1="13.97" x2="50.8" y2="20.32" width="0.4064" layer="1" curve="-90"/>
-<via x="48.26" y="22.86" extent="1-16" drill="0.6" shape="square"/>
-<wire x1="50.8" y1="20.32" x2="48.26" y2="22.86" width="0.4064" layer="1"/>
-<wire x1="45.72" y1="22.86" x2="48.26" y2="22.86" width="0.4064" layer="16"/>
-<wire x1="55.245" y1="13.97" x2="55.485" y2="13.97" width="0" layer="19" extent="1-1"/>
+<wire x1="45.72" y1="22.86" x2="45.72" y2="25.4" width="0.4064" layer="16"/>
+<wire x1="45.72" y1="25.4" x2="47.625" y2="24.13" width="0.4064" layer="1" curve="-90"/>
+<wire x1="47.625" y1="24.13" x2="47.625" y2="13.335" width="0.4064" layer="1"/>
+<wire x1="47.625" y1="13.335" x2="48.26" y2="12.7" width="0.4064" layer="1" curve="90"/>
+<wire x1="55.485" y1="13.97" x2="52.07" y2="13.335" width="0.4064" layer="1"/>
+<wire x1="52.07" y1="13.335" x2="48.26" y2="12.7" width="0.4064" layer="1"/>
+<via x="48.26" y="12.7" extent="1-16" drill="0.6" shape="square"/>
+<via x="45.72" y="25.4" extent="1-16" drill="0.6" shape="square"/>
 </signal>
 <signal name="N$8">
@@
 <wire x1="53.34" y1="7.62" x2="53.6194" y2="7.3406" width="0.4064" layer="16" curve="90"/>
 <wire x1="53.6194" y1="7.3406" x2="53.8988" y2="7.3406" width="0.4064" layer="16"/>
-<wire x1="45.72" y1="7.62" x2="53.34" y2="7.62" width="0.4064" layer="1"/>
+<wire x1="45.72" y1="6.35" x2="52.07" y2="6.35" width="0.4064" layer="1"/>
+<wire x1="52.07" y1="6.35" x2="53.34" y2="7.62" width="0.4064" layer="1" curve="90"/>
 <via x="53.34" y="7.62" extent="1-16" drill="0.6" shape="square"/>
 <wire x1="12.7" y1="15.24" x2="11.43" y2="15.24" width="0.4064" layer="1"/>
 <wire x1="11.43" y1="15.24" x2="11.43" y2="1.27" width="0.4064" layer="1"/>
 <wire x1="11.43" y1="1.27" x2="45.72" y2="1.27" width="0.4064" layer="1"/>
-<wire x1="45.72" y1="1.27" x2="45.72" y2="7.62" width="0.4064" layer="1"/>
+<wire x1="45.72" y1="1.27" x2="45.72" y2="6.35" width="0.4064" layer="1"/>
 </signal>
 <signal name="N$9">
@@
 </signal>
 <signal name="N$7">
-<wire x1="60.96" y1="25.4" x2="60.96" y2="26.67" width="0.4064" layer="16"/>
-<wire x1="60.96" y1="26.67" x2="20.32" y2="26.67" width="0.4064" layer="1"/>
-<via x="60.96" y="26.67" extent="1-16" drill="0.6" shape="square"/>
+<wire x1="50.8" y1="26.67" x2="20.32" y2="26.67" width="0.4064" layer="1"/>
 <contactref element="SW2" pad="3"/>
 <contactref element="R2" pad="1"/>
@@
 <wire x1="60.59" y1="22.86" x2="60.96" y2="22.86" width="0.4064" layer="16"/>
 <wire x1="60.96" y1="22.86" x2="60.96" y2="25.4" width="0.4064" layer="16"/>
+<wire x1="50.8" y1="26.67" x2="50.8" y2="25.4" width="0.4064" layer="1"/>
+<wire x1="50.8" y1="25.4" x2="53.975" y2="25.4" width="0.4064" layer="16"/>
+<wire x1="53.975" y1="25.4" x2="53.975" y2="24.765" width="0.4064" layer="16"/>
+<wire x1="53.975" y1="25.4" x2="60.4012" y2="25.1206" width="0" layer="19" extent="16-16"/>
+<via x="50.8" y="25.4" extent="1-16" drill="0.6" shape="square"/>
 </signal>
 <signal name="N$3">
@@
 <wire x1="45.72" y1="15.24" x2="45.72" y2="12.7" width="0.254" layer="16"/>
 </signal>
+<signal name="N$5">
+<via x="48.26" y="15.24" extent="1-16" drill="0.6" shape="square"/>
+</signal>
+<signal name="N$6">
+<via x="48.26" y="20.32" extent="1-16" drill="0.6" shape="square"/>
+</signal>
 </signals>

Commit message: update circuit diagram documents. fix D+ D- line.
Connections:
- net N$1: now also IC3.15; no longer IC3.16
- net N$2: now also IC3.16; no longer IC3.15
Routing:
- net N$2: track 23.9 -> 25.8 mm, vias 2 -> 1
- net N$1: track 27.7 -> 26.9 mm
Changed lines of the file:
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@@
 </signal>
 <signal name="N$1">
-<contactref element="IC3" pad="16"/>
 <contactref element="X1" pad="2"/>
 <wire x1="48.26" y1="10.16" x2="46.99" y2="11.43" width="0.4064" layer="1" curve="-90"/>
-<wire x1="46.99" y1="11.43" x2="46.99" y2="16.51" width="0.4064" layer="1"/>
-<wire x1="46.99" y1="16.51" x2="44.45" y2="20.32" width="0.4064" layer="1"/>
-<wire x1="44.45" y1="20.32" x2="44.45" y2="24.13" width="0.4064" layer="1"/>
-<wire x1="44.45" y1="24.13" x2="43.18" y2="25.4" width="0.4064" layer="1" curve="90"/>
-<wire x1="43.18" y1="25.4" x2="43.18" y2="22.86" width="0.4064" layer="16"/>
+<wire x1="46.99" y1="11.43" x2="46.99" y2="24.13" width="0.4064" layer="1"/>
+<wire x1="46.99" y1="24.13" x2="45.72" y2="25.4" width="0.4064" layer="1" curve="90"/>
 <wire x1="55.32" y1="13.335" x2="55.485" y2="13.17" width="0.4064" layer="1" curve="-90"/>
 <wire x1="48.26" y1="10.16" x2="52.945" y2="12.065" width="0.4064" layer="1"/>
 <wire x1="52.945" y1="12.065" x2="55.485" y2="13.17" width="0.4064" layer="1"/>
 <via x="48.26" y="10.16" extent="1-16" drill="0.6" shape="square"/>
-<via x="43.18" y="25.4" extent="1-16" drill="0.6" shape="square"/>
-</signal>
-<signal name="N$2">
+<via x="45.72" y="25.4" extent="1-16" drill="0.6" shape="square"/>
 <contactref element="IC3" pad="15"/>
-<contactref element="X1" pad="3"/>
 <wire x1="45.72" y1="22.86" x2="45.72" y2="25.4" width="0.4064" layer="16"/>
-<wire x1="45.72" y1="25.4" x2="47.625" y2="24.13" width="0.4064" layer="1" curve="-90"/>
-<wire x1="47.625" y1="24.13" x2="47.625" y2="13.335" width="0.4064" layer="1"/>
-<wire x1="47.625" y1="13.335" x2="48.26" y2="12.7" width="0.4064" layer="1" curve="90"/>
-<wire x1="55.485" y1="13.97" x2="52.07" y2="13.335" width="0.4064" layer="1"/>
-<wire x1="52.07" y1="13.335" x2="48.26" y2="12.7" width="0.4064" layer="1"/>
-<via x="48.26" y="12.7" extent="1-16" drill="0.6" shape="square"/>
-<via x="45.72" y="25.4" extent="1-16" drill="0.6" shape="square"/>
 </signal>
 <signal name="N$8">
@@
 <via x="48.26" y="20.32" extent="1-16" drill="0.6" shape="square"/>
 </signal>
+<signal name="N$2">
+<contactref element="IC3" pad="16"/>
+<contactref element="X1" pad="3"/>
+<wire x1="55.485" y1="13.97" x2="48.26" y2="13.97" width="0.4064" layer="1"/>
+<wire x1="48.26" y1="13.97" x2="48.26" y2="15.24" width="0.4064" layer="1"/>
+<wire x1="48.26" y1="15.24" x2="47.625" y2="15.24" width="0.4064" layer="1"/>
+<wire x1="47.625" y1="15.24" x2="47.625" y2="20.32" width="0.4064" layer="1"/>
+<wire x1="47.625" y1="20.32" x2="44.45" y2="20.32" width="0.4064" layer="1"/>
+<wire x1="44.45" y1="20.32" x2="44.45" y2="24.765" width="0.4064" layer="1"/>
+<wire x1="44.45" y1="24.765" x2="43.18" y2="25.4" width="0.4064" layer="1"/>
+<wire x1="43.18" y1="25.4" x2="43.18" y2="22.86" width="0.4064" layer="16"/>
+<via x="43.18" y="25.4" extent="1-16" drill="0.6" shape="square"/>
+</signal>
 </signals>
